Commit message: refactor: caster whell balance

File: description/robot_core.xacro (robot description, xacro)
@@ -9,8 +9,8 @@
     <xacro:property name="wheel_thickness" value="0.026"/>
     <xacro:property name="wheel_mass" value="0.05"/>
-    <xacro:property name="caster_wheel_radius" value="${wheel_radius}"/>
-    <xacro:property name="caster_wheel_mass" value="0.01"/>
-    <xacro:property name="caster_wheel_offset_x" value="${chassis_radius - caster_wheel_radius}"/>
-    <xacro:property name="caster_wheel_offset_z" value="${caster_wheel_radius/4}"/>
+    <xacro:property name="caster_wheel_radius" value="${wheel_radius+0.005}"/>
+    <xacro:property name="caster_wheel_mass" value="0.5"/>
+    <xacro:property name="caster_wheel_offset_x" value="${chassis_radius - caster_wheel_radius - 0.005}"/>
+    <xacro:property name="caster_wheel_offset_z" value="${caster_wheel_radius/6}"/>
     <material name="white">
         <color rgba="1 1 1 1" />

Commit message: refactor: caster wheel mass and offset

File: description/robot_core.xacro (robot description, xacro)
@@ -8,9 +8,9 @@
     <xacro:property name="wheel_radius" value="0.033"/>
     <xacro:property name="wheel_thickness" value="0.026"/>
-    <xacro:property name="wheel_mass" value="0.05"/>
+    <xacro:property name="wheel_mass" value="5"/>
     <xacro:property name="caster_wheel_radius" value="${wheel_radius+0.005}"/>
-    <xacro:property name="caster_wheel_mass" value="0.5"/>
+    <xacro:property name="caster_wheel_mass" value="50"/>
     <xacro:property name="caster_wheel_offset_x" value="${chassis_radius - caster_wheel_radius - 0.005}"/>
-    <xacro:property name="caster_wheel_offset_z" value="${caster_wheel_radius/6}"/>
+    <xacro:property name="caster_wheel_offset_z" value="${caster_wheel_radius/7}"/>
     <material name="white">
         <color rgba="1 1 1 1" />

Commit message: refactor: increase robot mass

File: description/robot_core.xacro (robot description, xacro)
@@ -4,11 +4,11 @@
     <xacro:property name="chassis_radius" value="0.1"/>
     <xacro:property name="chassis_thickness" value="0.05"/>
-    <xacro:property name="chassis_mass" value="1.0"/>
+    <xacro:property name="chassis_mass" value="10.0"/>
     <!-- Separator -->
     <xacro:property name="wheel_radius" value="0.033"/>
     <xacro:property name="wheel_thickness" value="0.026"/>
-    <xacro:property name="wheel_mass" value="5"/>
+    <xacro:property name="wheel_mass" value="50.0"/>
     <xacro:property name="caster_wheel_radius" value="${wheel_radius+0.005}"/>
-    <xacro:property name="caster_wheel_mass" value="50"/>
+    <xacro:property name="caster_wheel_mass" value="50.0"/>
     <xacro:property name="caster_wheel_offset_x" value="${chassis_radius - caster_wheel_radius - 0.005}"/>
     <xacro:property name="caster_wheel_offset_z" value="${caster_wheel_radius/7}"/>
