Commit message: chore: disable lidar visibility

File: description/lidar.xacro (robot description, xacro)
@@ -1,34 +1,34 @@
 <?xml version="1.0"?>
-<robot xmlns:xacro="http://www.ros.org/wiki/xacro" >
-    <xacro:property name="laser_foot_radius" value="0.01"/>
-    <xacro:property name="laser_foot_thickness" value="0.03"/>
-     <xacro:property name="laser_radius" value="0.025"/>
-    <xacro:property name="laser_thickness" value="0.02"/>
+<robot xmlns:xacro="http://www.ros.org/wiki/xacro">
+    <xacro:property name="laser_foot_radius" value="0.01" />
+    <xacro:property name="laser_foot_thickness" value="0.03" />
+    <xacro:property name="laser_radius" value="0.025" />
+    <xacro:property name="laser_thickness" value="0.02" />
     <joint name="laser_joint" type="fixed">
-        <parent link="chassis"/>
-        <child link="laser_frame"/>
-        <origin xyz="0 0 ${chassis_thickness + laser_foot_thickness}" rpy="0 0 0"/>
+        <parent link="chassis" />
+        <child link="laser_frame" />
+        <origin xyz="0 0 ${chassis_thickness + laser_foot_thickness}" rpy="0 0 0" />
     </joint>
     <link name="laser_frame">
         <visual>
             <geometry>
-                <cylinder radius="${laser_radius}" length="${laser_thickness}"/>
+                <cylinder radius="${laser_radius}" length="${laser_thickness}" />
             </geometry>
-            <material name="black"/>
+            <material name="black" />
         </visual>
         <visual>
-            <origin xyz="0 0 ${-laser_thickness}"/>
+            <origin xyz="0 0 ${-laser_thickness}" />
             <geometry>
-                <cylinder radius="${laser_foot_radius}" length="${laser_foot_thickness}"/>
+                <cylinder radius="${laser_foot_radius}" length="${laser_foot_thickness}" />
             </geometry>
-            <material name="black"/>
+            <material name="black" />
         </visual>
         <collision>
             <geometry>
-                <cylinder radius="${laser_radius}" length="${laser_thickness}"/>
+                <cylinder radius="${laser_radius}" length="${laser_thickness}" />
             </geometry>
         </collision>
         <xacro:inertial_cylinder mass="0.1" length="${laser_thickness}" radius="${laser_radius}">
-            <origin xyz="0 0 0" rpy="0 0 0"/>
+            <origin xyz="0 0 0" rpy="0 0 0" />
         </xacro:inertial_cylinder>
     </link>
@@ -37,5 +37,5 @@
         <sensor name="laser" type="ray">
             <pose> 0 0 0 0 0 0 </pose>
-            <visualize>true</visualize>
+            <visualize>false</visualize>
             <update_rate>20</update_rate>
             <always_on>1</always_on>
@@ -64,6 +64,6 @@
                 </noise>
             </ray>
-           <plugin name="laser_controller" filename="libgazebo_ros_ray_sensor.so">
-                 <ros>
+            <plugin name="laser_controller" filename="libgazebo_ros_ray_sensor.so">
+                <ros>
                     <argument>~/out:=lidar_scan</argument>
                 </ros>
